File: NixieDriver_mx.brd (EAGLE design)
At the start: 67 x 55.9 mm, 18 parts, among them IC1 PIC18F2550_28DIP, IC2 74141N, Q1 20MHz, T1 BF420, T2 BF420, T3 BF420, X1 USB-B-H

Commit message: Dump current status from laptop
Parts:
- added R10, R4, R7: 3.3k, rcl:0207/7
- added R2, R5, R8: 3.3k, rcl:0207/2V
- added R3, R6, R9: 100k, rcl:0207/5V
- added T4, T6: BF420, transistor-neu-to92:TO92-ECB
- added T5: BF421, transistor-neu-to92:TO92-ECB
- T1: device transistor:TO92-BCE -> transistor-neu-to92:TO92-ECB
- T2, T3: value BF420 -> BF421; device transistor:TO92-BCE -> transistor-neu-to92:TO92-ECB
- moved T1 16.5 mm to (66.0, 36.8), turned to 0 degrees
- moved T2 13.1 mm to (66.0, 43.2)
- moved T3 8.13 mm to (54.6, 43.2)
- moved PAD4 6.48 mm to (61.0, 50.8)
- moved PAD3 6.48 mm to (69.8, 50.8)
- moved IC2 3.59 mm to (45.7, 15.2)
- moved JP3 2.54 mm to (57.1, 16.5)
- moved PAD2 2.54 mm to (39.4, 49.5)
Connections:
- new net N$10: R9.2, T5.B, T6.C
- new net N$11: R10.1, T6.E
- new net N$12: R8.1, T6.B
- new net N$4: R3.2, T1.C, T2.B
- new net N$5: R2.1, T1.B
- new net N$6: R4.1, T1.E
- new net N$7: R6.2, T3.B, T4.C
- new net N$8: R7.1, T4.E
- new net N$9: R5.1, T4.B
- net +HV: now also R3.1, R6.1, R9.1, T2.E, T3.E, T5.E; no longer T1.C, T2.C, T3.C
- net DIG1_ANODE: now also JP3.8, T2.C; no longer JP3.4, T1.E
- net DIG1_GATE: now also R2.2; no longer T1.B
- net DIG2_ANODE: now also T3.C; no longer T2.E
- net DIG2_GATE: now also R5.2; no longer T2.B
- net DIG3_ANODE: now also JP3.4, T5.C; no longer JP3.8, T3.E
- net DIG3_GATE: now also R8.2; no longer T3.B
- net GND: now also R10.2, R4.2, R7.2
Routing:
- net N$5: track 0.00 -> 39.3 mm
- net DIG3_GATE: track 36.5 -> 3.81 mm
- net N$9: track 0.00 -> 27.9 mm
- net DIG2_GATE: track 30.9 -> 3.81 mm
- net DIG1_GATE: track 25.0 -> 3.81 mm
- net DIG1_ANODE: track 19.8 -> 39.3 mm
- net GND: track 168.3 -> 187.1 mm
- net DIG3_ANODE: track 20.7 -> 38.2 mm, vias 0 -> 2
- net N$12: track 0.00 -> 16.6 mm
- net DIG2_ANODE: track 20.0 -> 33.7 mm, vias 0 -> 2
- net N$7: track 0.00 -> 7.62 mm
- net N$10: track 0.00 -> 7.62 mm
- net N$4: track 0.00 -> 7.62 mm
- net +HV: track 25.1 -> 31.7 mm
- net N$8: track 0.00 -> 4.34 mm
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Other:
- board size 67 x 55.9 mm -> 74.6 x 55.9 mm
